Commit message: Update

File: workspace/src/robot_scene/urdf/robot_model.xacro (robot description, xacro)
@@ -2,5 +2,4 @@
 <robot name="robot" xmlns:xacro="http://www.ros.org/wiki/xacro">
     <xacro:include filename="materials.xacro" />
-    <xacro:include filename="robot_model.gazebo" />
     <xacro:include filename="wheel.xacro" />
     <xacro:include filename="inertial.xacro" />
@@ -24,4 +23,12 @@
         </joint>
     </ros2_control>
+    <gazebo>
+        <plugin filename="gz_ros2_control-system"
+        name="gz_ros2_control::GazeboSimROS2ControlPlugin">
+            <parameters>
+            $(find robot_scene)/config/diff_control.yaml
+            </parameters>
+        </plugin>
+    </gazebo>
     <link name='base_link'>
         <origin xyz="0.0 0.0 0.1" rpy="0.0 0 0.0"/>
@@ -116,7 +123,5 @@
         <visual name='lidar_visual'>
             <origin xyz="0 0 0" rpy=" 0 0 0"/>
-            <geometry>
-                <box size="0.05 0.05 0.05"/>
-            </geometry>
+            <geometry><box size="0.05 0.05 0.05"/></geometry>
             <material name="red"/>
         </visual>
@@ -130,7 +135,5 @@
         <collision>
             <origin xyz="0 0 0" rpy="0 0 0"/>
-                <geometry>
-                    <box size="0.05 0.05 0.05"/>
-                </geometry>
+                <geometry><box size="0.05 0.05 0.05"/></geometry>
         </collision>
     </link>
